Commit message: 完整定位导航一版

File: src/robot_base/urdf/four_diff.urdf (robot description, URDF)
Before this commit: robot robotcar, 8 links, 7 joints
Joints:
- joint livox_joint: origin xyz=0.34 0 0.3 rpy=0 -0.785398 0 -> xyz=0.34 0 0.3 rpy=0 0 0

File: src/robot_base/urdf/four_diff.xacro (robot description, xacro)
@@ -51,5 +51,5 @@
     <parent link="base_link"/>
     <child link="livox_frame"/>
-    <origin xyz="${body_length/2} 0 ${body_height}" rpy="0 -0.785398 0"/> <!-- 绕 Y 轴向上倾斜 45 度补偿物理向下角度，使scan水平 -->
+    <origin xyz="${body_length/2} 0 ${body_height}" rpy="0 0 0"/> <!-- 数据已预处理为水平，此处设为0 -->
   </joint>
   <!-- Wheels Macro -->
