Commit message: feat: add route navigation, waypoint editor, and related improvements

File: src/robot_base/urdf/robotcar.urdf (robot description, URDF)
Before this commit: robot robotcar, 15 links, 14 joints
Links:
- removed link camera_link
- removed link camera_optical_frame
- removed link fl_caster_caster_link
- removed link fr_caster_caster_link
- removed link front_right_laser
- removed link front_right_lidar_hollow_ring
- removed link rear_left_laser
- removed link rear_left_lidar_hollow_ring
- removed link rl_caster_caster_link
- removed link rr_caster_caster_link
- added link livox_frame; visual cylinder length=0.05 radius=0.03
- added link rear_caster_link, mass 0.5; collision sphere radius=0.04; visual sphere radius=0.04
- link base_link: mass 50 -> 20.0; geometry collision box size=0.68 0.33 0.3; visual box size=0.68 0.33 0.3
- link imu_link: mass 0.01 -> None; geometry visual box size=0.02 0.02 0.01
- link left_wheel_link: geometry collision cylinder length=0.03 radius=0.08; visual cylinder length=0.03 radius=0.08
- link right_wheel_link: geometry collision cylinder length=0.03 radius=0.08; visual cylinder length=0.03 radius=0.08
Joints:
- removed joint camera_joint
- removed joint camera_optical_joint
- removed joint fl_caster_caster_joint
- removed joint fr_caster_caster_joint
- removed joint front_right_laser_joint
- removed joint front_right_lidar_hollow_joint
- removed joint rear_left_laser_joint
- removed joint rear_left_lidar_hollow_joint
- removed joint rl_caster_caster_joint
- removed joint rr_caster_caster_joint
- added joint livox_joint: type fixed, parent base_link, child livox_frame, origin xyz=0.34 0.0 0.15 rpy=0 0.785398 0
- added joint rear_caster_joint: type fixed, parent base_link, child rear_caster_link, origin xyz=-0.22 0 -0.16 rpy=0 0 0
- joint base_joint: origin xyz=0 0 0.047 rpy=0 0 0 -> xyz=0 0 0.2 rpy=0 0 0
- joint left_wheel_joint: limit effort=10.0 velocity=10.0 -> (none); origin xyz=0 0.26499999999999996 0.0 rpy=0 0 0 -> xyz=0.22 0.13 -0.12000000000000001 rpy=0 0 0
- joint right_wheel_joint: limit effort=10.0 velocity=10.0 -> (none); origin xyz=0 -0.26499999999999996 0.0 rpy=0 0 0 -> xyz=0.22 -0.13 -0.12000000000000001 rpy=0 0 0

File: src/robot_base/urdf/robotcar.xacro (robot description, xacro)
@@ -15,4 +15,5 @@
   <xacro:property name="wheel_radius" value="0.08"/>
   <xacro:property name="wheel_length" value="0.03"/>
+  <xacro:property name="caster_radius" value="0.04"/>
   <!-- 轮距参数 -->
   <!-- 轮子边缘外切线距离前后4cm -->
@@ -109,17 +110,17 @@
   <xacro:wheel_link name="right" parent_link="base_link"
                     x_offset="${wheelbase_half}" y_offset="-${track_half}" z_offset="${wheel_z_offset}"/>
-  <!-- 左后轮 (从动/Mimic) -->
-  <link name="rear_left_wheel_link">
-    <visual>
-      <origin xyz="0 0 0" rpy="${M_PI/2} 0 0"/>
-      <geometry>
-        <cylinder length="${wheel_length}" radius="${wheel_radius}"/>
+  <!-- ======================== 后置万向轮 ======================== -->
+  <link name="rear_caster_link">
+    <visual>
+      <origin xyz="0 0 0" rpy="0 0 0"/>
+      <geometry>
+        <sphere radius="${caster_radius}"/>
       </geometry>
       <material name="black"/>
     </visual>
     <collision>
-      <origin xyz="0 0 0" rpy="${M_PI/2} 0 0"/>
-      <geometry>
-        <cylinder length="${wheel_length}" radius="${wheel_radius}"/>
+      <origin xyz="0 0 0" rpy="0 0 0"/>
+      <geometry>
+        <sphere radius="${caster_radius}"/>
       </geometry>
     </collision>
@@ -129,38 +130,15 @@
     </inertial>
   </link>
-  <joint name="rear_left_wheel_joint" type="continuous">
+  <joint name="rear_caster_joint" type="fixed">
     <parent link="base_link"/>
-    <child link="rear_left_wheel_link"/>
-    <origin xyz="-${wheelbase_half} ${track_half} ${wheel_z_offset}" rpy="0 0 0"/>
-    <axis xyz="0 1 0"/>
-    <mimic joint="left_wheel_joint" multiplier="1.0" offset="0.0"/>
-  </joint>
-  <!-- 右后轮 (从动/Mimic) -->
-  <link name="rear_right_wheel_link">
-    <visual>
-      <origin xyz="0 0 0" rpy="${M_PI/2} 0 0"/>
-      <geometry>
-        <cylinder length="${wheel_length}" radius="${wheel_radius}"/>
-      </geometry>
-      <material name="black"/>
-    </visual>
-    <collision>
-      <origin xyz="0 0 0" rpy="${M_PI/2} 0 0"/>
-      <geometry>
-        <cylinder length="${wheel_length}" radius="${wheel_radius}"/>
-      </geometry>
-    </collision>
-    <inertial>
-      <mass value="0.5"/>
-      <inertia ixx="0.001" ixy="0" ixz="0" iyy="0.001" iyz="0" izz="0.001"/>
-    </inertial>
-  </link>
-  <joint name="rear_right_wheel_joint" type="continuous">
-    <parent link="base_link"/>
-    <child link="rear_right_wheel_link"/>
-    <origin xyz="-${wheelbase_half} -${track_half} ${wheel_z_offset}" rpy="0 0 0"/>
-    <axis xyz="0 1 0"/>
-    <mimic joint="right_wheel_joint" multiplier="1.0" offset="0.0"/>
-  </joint>
+    <child link="rear_caster_link"/>
+    <origin xyz="-${wheelbase_half} 0 ${caster_radius - base_link_z_offset}" rpy="0 0 0"/>
+  </joint>
+  <!-- Gazebo simulation: Frictionless caster -->
+  <gazebo reference="rear_caster_link">
+    <mu1>0.0</mu1>
+    <mu2>0.0</mu2>
+    <material>Gazebo/Black</material>
+  </gazebo>
   <!-- ======================== 传感器 ======================== -->
   <!-- Lidar: Mid-360 -->
